File: pcb/pcb.kicad_sch (KiCad schematic)
At the start: 104 parts

Commit message: battery power
Parts:
- removed C? (x2): 0.1uF, symbol Device:C_Small
- added BT?: Li-ion, symbol Device:Battery_Cell
- added C? (x5): 10uF, symbol Device:C_Small
- added C? (x3): 0.1uF, symbol Device:C_Small
- added C?: 100uF, symbol Device:C_Polarized_Small
- added D? (x3): 1N5822, Diode_THT:D_DO-201AD_P15.24mm_Horizontal, symbol Diode:1N5822
- added L?: 4.7uH, symbol Device:L_Small
- added LS?: Speaker, symbol Device:Speaker
- added R?: 330k, symbol Device:R
- added R?: 47k, symbol Device:R
- added R? (x2): 10k, symbol Device:R
- added R? (x2): 100k, symbol Device:R
- added SW?: on/off, symbol Switch:SW_SPST
Connections:
- net +12V: now also C?.1, C?.1, D?.1 (K), R?.1
- net -12V: now also C?.1, C?.2, D?.2 (A)
- net 10: now also R?.2
- net GND: now also U?.2 (GND), U?.7 (V-), BT?.2 (-), C?.1, C?.1, C?.2, C?.2, C?.2, C?.2, C?.2, C?.2, D?.1 (K), R?.2, SW?.2 (B)
- net at U?.1 (SW): now also D?.2 (A), L?.2, R?.2
- net at U?.3 (FB): now also R?.1, R?.2
- net 1: now reaches U?.4 (EN)
- net 1: now also U?.1 (SHUTDOWN), R?.1, SW?.1 (A)
- net +3V8: now reaches U?.5 (VIN)
- net +3V8: now also U?.6 (V+), BT?.1 (+), C?.1, C?.1, C?.1, L?.1, R?.2
- net at U?.2 (BYPASS): now also U?.3 (IN+), C?.2
- net at U?.4 (IN-): now also R?.1, R?.2
- net at U?.5 (VoutA): now also LS?.1, R?.1
- net at U?.8 (VoutB): now also LS?.2
- new net: C?.1, R?.1
- new net: C?.2, D?.1 (K), D?.2 (A)
Other:
- moved on the sheet: U?, U?E
